File: preamp/preamp.sch (KiCad schematic (older format))
At the start: 19 parts, among them J1 Earth, J2 Filament, J3 B+, J4 CH1, J5 CH2, J6 CH2 volume pot (4M), J7 CH1 volume pot (4M), J8 Audio Out

Commit message: Hacking for Feb 1st, 2019
Parts:
- removed C4: 0.001uF 400V, symbol Device:C
- added C?: 10uF 400V, symbol Device:C
- J4: value CH1 -> CH 2
- J5: value CH2 -> CH1
- J6: value CH2 volume pot (4M) -> CH1 volume pot (4M)
- J7: value CH1 volume pot (4M) -> CH2 volume pot (4M)
Connections:
- net Earth: now also C?.2
- net at R2.1, R3.2, R4.1: now also C?.1
- net fil_a renamed f1
- net f1: now also V1.9; no longer V1.5-UB
- net fil_b renamed f2
- net f2: now also V1.5-UB; no longer V1.9
Other:
- moved on the sheet: C1, C2, C3, J1, J2, J3, J4, J5, J6, J8, R1, R4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
