File: actual/actual.sch (KiCad schematic (older format))
At the start: 192 parts, among them J1 in_lo, J10 effect return, J11 PWR, J12 el84, J13 V_power, J14 RG, J15 RC, J16 105-1103-001, J17 105-1103-001, J18 105-1103-001, J2 in_hi, J3 IEC_SOCKET, J4 Tank IN, J5 Audio Out, J6 Reverb Footswitch, J7 tremolo footswitch, J8 Tank OUT, J9 effect send, SW2 A.C., SW3 STANDBY, T1 78633, T2 68348, T3 Transformer_125ASE

Commit message: Major renovations
* Replace phase inverter with op-amp phase inverter.
* Create a dual rail DC op-amp power supply driven off the filament supply lines.
* Replace 7027 tubes with 6L6GC tubes.
* Add switched IEC outlet.
Parts:
- removed C8: 0.047 400V, symbol Device:C
- removed C9: 0.1uF, symbol Device:C
- removed J16, J17, J18: 105-1103-001, digikey-footprints:Test_Jack_Horiz, symbol dk_Banana-and-Tip-Connectors-Jacks-Plugs:105-1103-001
- removed R19: 68K, symbol Device:R
- removed R20, R22: 470K, symbol Device:R
- removed R21: 470, symbol Device:R
- removed R23: 4.7K, symbol Device:R
- removed R24: 82K, symbol Device:R
- removed R25: 100K, symbol Device:R
- removed RV10: 100, symbol Device:R_POT
- removed TP26, TP27, TP28: TestPoint, symbol Connector:TestPoint
- removed V3: 12AX7, Valve:Valve_ECC-83-1, symbol local:12AX7
- added C43: 1000uF, symbol Device:CP
- added C44: 0.047uF, symbol Device:C
- added C45, C46: .1uF, symbol Device:C
- added C47: 0.022uF, symbol Device:C
- added C48: 0.22uF, symbol Device:C
- added D8: BU1006, symbol Device:D_Bridge_+AA-
- added J16: MDL_AC, symbol Connector:Screw_Terminal_01x02
- added J17: MDL_PWR, symbol Connector:Screw_Terminal_01x04
- added J18, J19: PI_PWR, symbol Connector:Screw_Terminal_01x04
- added J?: Switched power, symbol local:Conn_IEC_Power
- added PS1: IH0515D, Converter_DCDC:Converter_DCDC_XP_POWER-IHxxxxD_THT, symbol Converter_DCDC:IH0515D
- added R65: 100K, symbol Device:R
- added R67, R77, R78: 1K, symbol Device:R
- added R68, R70: 20K, symbol Device:R
- added R69: 18K, symbol Device:R
- added R71, R72: 300, symbol Device:R
- added R73, R74: 1M, symbol Device:R
- added R75, R76: 220K, symbol Device:R
- added U1: OPA2134PA, digikey-footprints:DIP-8_W7.62mm, symbol dk_Linear-Amplifiers-Instrumentation-OP-Amps-Buffer-Amps:OPA2134PA
- added V10: ECC803S, Valve:Valve_ECC-83-1, symbol local:12AX7
- C10, C11: value 0.1uF 400V -> 0.1uF
- C20: value 47nF -> 0.047uF
- R28: value 100K -> 82K
- V4, V5: value 7027A -> 6L6GC
- V9: value EL84 -> EL844
Connections:
- net B+: now also R75.1, R76.1
- net Earth: now also C45.2, C46.2, J17.2 (Pin_2), J18.2 (Pin_2), J18.3 (Pin_3), PS1.6 (0V), R73.2, R74.2, R77.1, R78.1, U1.3, U1.5
- net V2: now also R29.2, R30.1
- net f1: now also D8.2 (~~), J16.1 (Pin_1), V10.5 (f), V10.9 (f)
- net f2: now also D8.3 (~~), J16.2 (Pin_2), V10.4 (f), V10.9 (f)
- net at J3.3 (N), T1.2 (AB): now also J?.2 (AC_N)
- net at F1.2, SW2.2 (B): now also J?.1 (AC_P)
- net at C11.2: now also R76.2, V10.1 (a)
- net at C11.1, TP30.1, V5.5 (G): now also R26.1; no longer R26.2
- net pi_in: now reaches RV7.2, TP25.1
- net pi_in: now also C44.2, J19.1 (Pin_1)
- net at R28.1: now also J5.T, T2.5 (S2), TP34.1
- net at C10.2: now also R75.2, V10.6 (a)
- net at C14.1, R27.2, RV5.2: now also R26.2; no longer R26.1
- net at C38.2, RV9.2: now also R65.1
- net at C38.1, RV7.3: now also R65.2
- new net: R68.2, R69.1, R71.2, U1.1
- new net: R68.1, R70.2, U1.6
- new net: R70.1, R72.2, U1.7
- new net: C44.1, R67.2
- new net: C43.1, D8.1 (+), PS1.3 (+Vin)
- new net: C43.2, D8.4 (-), PS1.1 (-Vin)
- new net: R77.2, V10.8 (k)
- new net: C48.1, R74.1, V10.2 (g)
- new net: R78.2, V10.3 (k)
- new net: C47.1, R73.1, V10.7 (g)
- new net +15V: C45.1, J17.3 (Pin_3), J18.1 (Pin_1), PS1.5 (+Vout), U1.8 (V+), U1.8 (V+)
- new net -15V: C46.1, J17.1 (Pin_1), J18.4 (Pin_4), PS1.4 (-Vout), U1.4 (V-), U1.4 (V-)
- new net pi_a: C47.2, J19.3 (Pin_3), R71.1
- new net pi_b: C48.2, J19.4 (Pin_4), R72.1
- new net pi_fb: J19.2 (Pin_2), R28.2, R67.1, R69.2, U1.2
Other:
- moved on the sheet: C14, C15, C16, C17, C18, C19, C20, J7, R26, R27, R28, R34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

Commit message: add bypass capacitors to tube gain stage following op-amp phase inverter.
Parts:
- added C42, C9: 27uF, symbol Device:CP
- added C8: 0.02uF, symbol Device:C
- added R19: 4.7K, symbol Device:R
- gave numbers to parts that had none: 1
Connections:
- net Earth: now also C42.2, C9.2
- net rc1: now also C8.2; no longer J14.4 (Pin_4), R10.1, V7.7 (g)
- net at R77.2, V10.8 (k): now also C9.1
- net at R78.2, V10.3 (k): now also C42.1
- new net: C8.1, R19.2
- new net rg4: J14.4 (Pin_4), R10.1, R19.1, V7.7 (g)
Changed lines of the file:
@@
 	16800 7050 17050 7050
 Connection ~ 16600 7600
-Wire Wire Line
-	1100 4950 1100 8550
-Wire Wire Line
-	1100 8550 2850 8550
-Connection ~ 1100 8550
-Wire Wire Line
-	1100 8550 1100 10950
 $Comp
-L local:Conn_IEC_Power J?
+L local:Conn_IEC_Power J20
 U 1 1 62FBD204
 P 1650 14400
-F 0 "J?" H 1531 14725 50  0000 C CNN
+F 0 "J20" H 1531 14725 50  0000 C CNN
 F 1 "Switched power" H 1531 14634 50  0000 C CNN
 F 2 "" H 1855 14400 50  0001 C CNN
@@
 	2200 14300 1750 14300
 Connection ~ 2200 13250
+Wire Wire Line
+	1100 4950 1100 8550
+$Comp
+L Device:C C8
+U 1 1 5F4F92B9
+P 1500 8550
+F 0 "C8" V 1248 8550 50  0000 C CNN
+F 1 "0.02uF" V 1339 8550 50  0000 C CNN
+F 2 "" H 1538 8400 50  0001 C CNN
+F 3 "~" H 1500 8550 50  0001 C CNN
+	1    1500 8550
+	0    1    1    0
+$EndComp
+$Comp
+L Device:R R19
+U 1 1 5F5352DE
+P 2150 8550
+F 0 "R19" V 1943 8550 50  0000 C CNN
+F 1 "4.7K" V 2034 8550 50  0000 C CNN
+F 2 "" V 2080 8550 50  0001 C CNN
+F 3 "~" H 2150 8550 50  0001 C CNN
+	1    2150 8550
+	0    1    1    0
+$EndComp
+Wire Wire Line
+	2850 8550 2300 8550
+Wire Wire Line
+	2000 8550 1650 8550
+Wire Wire Line
+	1350 8550 1100 8550
+Connection ~ 1100 8550
+Wire Wire Line
+	1100 8550 1100 10950
+Wire Notes Line
+	12600 3700 12600 8650
+Wire Notes Line
+	12600 8650 16500 8650
+Wire Notes Line
+	16500 8650 16500 3700
+Wire Notes Line
+	16500 3700 12600 3700
+$Comp
+L Device:CP C9
+U 1 1 5F7C8B82
+P 16300 5750
+F 0 "C9" H 16418 5796 50  0000 L CNN
+F 1 "27uF" H 16418 5705 50  0000 L CNN
+F 2 "" H 16338 5600 50  0001 C CNN
+F 3 "~" H 16300 5750 50  0001 C CNN
+	1    16300 5750
+	1    0    0    -1
+$EndComp
+Wire Wire Line
+	16000 5700 16000 5600
+Wire Wire Line
+	16000 5600 16300 5600
+Connection ~ 16000 5600
+$Comp
+L power:Earth #PWR037
+U 1 1 5F80C7A1
+P 16300 6000
+F 0 "#PWR037" H 16300 5750 50  0001 C CNN
+F 1 "Earth" H 16300 5850 50  0001 C CNN
+F 2 "" H 16300 6000 50  0001 C CNN
+F 3 "~" H 16300 6000 50  0001 C CNN
+	1    16300 6000
+	1    0    0    -1
+$EndComp
+Wire Wire Line
+	16300 6000 16300 5900
+$Comp
+L Device:CP C42
+U 1 1 5F84D89F
+P 16300 8200
+F 0 "C42" H 16418 8246 50  0000 L CNN
+F 1 "27uF" H 16418 8155 50  0000 L CNN
+F 2 "" H 16338 8050 50  0001 C CNN
+F 3 "~" H 16300 8200 50  0001 C CNN
+	1    16300 8200
+	1    0    0    -1
+$EndComp
+Wire Wire Line
+	16000 8050 16300 8050
+$Comp
+L power:Earth #PWR057
+U 1 1 5F84D8AA
+P 16300 8450
+F 0 "#PWR057" H 16300 8200 50  0001 C CNN
+F 1 "Earth" H 16300 8300 50  0001 C CNN
+F 2 "" H 16300 8450 50  0001 C CNN
+F 3 "~" H 16300 8450 50  0001 C CNN
+	1    16300 8450
+	1    0    0    -1
+$EndComp
+Wire Wire Line
+	16300 8450 16300 8350
+Connection ~ 16000 8050
 $EndSCHEMATC
