File: actual/actual.sch (KiCad schematic (older format))
At the start: 207 parts, among them J1 in_lo, J10 effect return, J11 PWR, J12 el84, J13 V_power, J14 RG, J15 RC, J16 MDL_AC, J17 MDL_PWR, J18 PI_PWR, J19 PI_PWR, J2 in_hi, J20 Switched power, J3 IEC_SOCKET, J4 Tank IN, J5 Audio Out, J6 Reverb Footswitch, J7 tremolo footswitch, J8 Tank OUT, J9 effect send, SW2 A.C., SW3 STANDBY, T1 78633, T2 68348, T3 Transformer_125ASE, U1 OPA2134PA

Commit message: fixing bugs
Parts:
- removed C37: 10n, symbol Device:C
- removed C38: 330pF, symbol Device:C
- removed R62, R63: 360K, symbol Device:R
- removed R65: 100K, symbol Device:R
- removed RV9: 50kB, symbol Device:R_POT
- removed TP23: TestPoint, symbol Connector:TestPoint
- added R20: 36K, symbol Device:R
- added R21: 820k, symbol Device:R
- R28: value 82K -> 200K
- R69: value 18K -> 20K
Connections:
- wire segments 485 -> 477
Other:
- moved on the sheet: C2, C27, C28, C36, C39, J1, J2, R1, R14, R2, R28, R3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

Commit message: evening hacking
fix more buzz by rewiring the V2 socket.
Install RG-178 coax on most of the signal path. Reduce a bit more noise.
Remove the preamp circuit all together. Going to work on designing a better sounding one that handles overdrive better.
Debbug the reverb mix knob setting oscillation issues.
Parts:
- removed C41: 0.001uF 630V, symbol Device:C
- removed R1: 68K, symbol Device:R
- removed R60: 1K, symbol Device:R
- removed TP24: TestPoint, symbol Connector:TestPoint
- added C?: 0.1uF 400V, symbol Device:C
- added R?: 68K, symbol Device:R
- added S?: tone bypass, symbol local:SW_SPDT
- C34: value 1uF -> 270uF
- C4: value 0.02uF 400V -> 0.1uF 400V
- J20: symbol local:Conn_IEC_Power -> actual-rescue:Conn_IEC_Power-local
Connections:
- wire segments 477 -> 457
Other:
- note added: "2nd volume knob"
- note added: "370V"
- note added: "400V"
- note added: "Input that bypasses preamp"
- note added: "Main Input"
- moved on the sheet: C1, C2, C27, C28, C39, C40, J1, J10, J2, J9, R11, R13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

Commit message: build a new preamp
having both 12AX7 and EF86 as switchable option for first stage.
Parts:
- removed C40: 0.001uF 630V, symbol Device:C
- removed C?: 0.1uF 400V, symbol Device:C
- removed S?: tone bypass, symbol local:SW_SPDT
- removed TP21: TestPoint, symbol Connector:TestPoint
- added C37: C, symbol Device:C
- added C38: 0.1uF 400V, symbol Device:C
- added C40: 10uF 400V, symbol Device:CP
- added J21, J23: PWR, symbol Connector:Screw_Terminal_01x02
- added J22: PG, symbol Connector:Screw_Terminal_01x04
- added R22: 220K, symbol Device:R
- added R23: 1M, symbol Device:R
- added R24: 10K 1W, symbol Device:R
- added RV9: 20K, symbol Device:R_POT
- added TP23, TP24: TestPoint, symbol Connector:TestPoint
- added V3: EF86, Valve:Valve_Noval_P, symbol local:EF86
- C1: value 270uF 16V -> 100uF
- C2: value 0.02uF 400V -> 0.1uF 400V
- C28: value 1uF 16V -> 100uF
- R11: value 100K -> 820
- R3: value 1M -> 68K
- R47: value 2.7K -> 820
- R7: value 820 -> 1M
- R75, R76: value 220K -> 100K
- R8: value 220K 1/2W -> 100K
- R9: value 100K 1/2W -> 100K
- gave numbers to parts that had none: 1
Connections:
- net B+: now also J21.1 (Pin_1), J23.1 (Pin_1), R24.2; no longer R13.1, TP16.1, V2.1 (a)
- net Earth: now also R11.2, C37.2, C40.2, J22.1 (Pin_1), RV9.1, V3.7,2 (S)
- net V1BC: now reaches C28.1, R47.1, TP5.1, V1.3 (k)
- net V1BC: now also J22.3 (Pin_3)
- net at C27.1, C39.1, R14.1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: now also J21.2 (Pin_2), R22.1, R23.1; no longer TP2.1
- net at RV1.3, TP8.1: now also S1.1; no longer C2.1
- net at R9.1: now also V1.6 (a), C38.2
- net at J1.TN, TP14.1: now also C38.1; no longer C4.1
- net at C4.2: now also R22.2, V3.6 (A); no longer V1.6 (a)
- net at R11.1: now also C1.1, TP2.1, V3.3 (K), V3.8 (G3)
- net at J2.T, R2.2: now also R3.2; no longer R59.1
- net at R2.1, V1.2 (g): now also R3.1, R59.1, R7.1, V3.9 (G1)
- net at S1.2: now also C4.1
- net at S1.3: now also C2.1
- net at RV1.2: now also V1.7 (g)
- net at RV3.2: now also J9.T
- net V1AC: now reaches V1.8 (k)
- net V1AC: now also TP10.1, J22.2 (Pin_2), RV9.2
- net at C48.1, R74.1, V10.2 (g): now also TP24.1
- net at C47.1, R73.1, V10.7 (g): now also TP23.1
- new net: C40.1, J23.2 (Pin_2), R13.1, R24.1, TP16.1, V2.1 (a)
- new net: C37.1, R23.2, V3.1 (G2)
Other:
- note added: "1.45V"
- note added: "216V"
- note added: "340V"
- note added: "Set to 10K"
- moved on the sheet: C10, C11, C12, C13, C14, C15, C16, C17, C18, C19, C2, C20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

Commit message: weekend hacking
Parts:
- removed R20: 36K, symbol Device:R
- removed R21: 820k, symbol Device:R
- added C41: 0.001uF 630V, symbol Device:C
- added RV10: 1M, symbol Device:R_Potentiometer
- added SW1: SW_DPDT_x2, symbol Switch:SW_DPDT_x2
- added TR1: 107V, symbol Transformer:TRANSF5
- C1, C12, C13, C28, C29, C33, C34, C35, C40, C42, C43, C9: symbol Device:CP -> actual-rescue:CP-Device
- C17: value 0.02uF -> 0.047uF; footprint 0.02uF -> (none)
- C20, C44: value 0.047uF -> 0.1uF
- L1: symbol Device:L_Core_Ferrite -> actual-rescue:L_Core_Ferrite-Device
- R9: value 100K -> 220K
- RV1, RV2, RV3, RV4, RV5, RV6, RV7, RV8, RV9: symbol Device:R_POT -> actual-rescue:R_POT-Device
Connections:
- net B+: now also V6.1 (a); no longer V6.6 (a)
- net Earth: now also RV10.3, TR1.3, TR1.4
- net pi_in: now also R1.2, RV7.2; no longer C44.2, R1.1
- net at C27.1, C39.1, J21.2 (Pin_2)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: now also C41.1
- net at C38.2, R9.1, V1.6 (a): now also C41.2
- net at RV7.3: now also RV10.2
- net at C36.1: now also RV10.1
- net at R34.1, R35.1: now also V6.3 (k); no longer V6.8 (k)
- net at C17.2, R36.1: now also V6.2 (g), V6.6 (a); no longer V6.1 (a), V6.7 (g)
- net at C16.1, R37.2, R38.1: now also V6.8 (k); no longer V6.3 (k)
- net at C19.2, R39.1: now also V6.7 (g); no longer V6.2 (g)
- new net: C44.2, R1.1
- new net: SW1.3 (C), TR1.1
- new net: SW1.6 (C), TR1.6
- no-connect marks 1 -> 3
Other:
- note added: "Reverb\nVolume"
- note added: "Set to 5K"
- note removed: "Set to 10K"
- moved on the sheet: C10, C11, C14, C15, C16, C17, C18, C19, C42, C44, C45, C46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
